File: CanSat/CanSat.kicad_pcb (KiCad board)
At the start: 2 copper layers, 78 parts, among them J1 XLR3_Switched, J10 Conn_01x02_Male, J11 Conn_01x02_Male, J12 Conn_01x02_Male, J13 Conn_01x02_Male, J14 Conn_01x02_Male, J2 Conn_01x04_Male, J3 Conn_01x02_Male, J4 Conn_01x02_Male, J5 Conn_01x02_Male, J6 Conn_01x02_Male, J7 Conn_01x02_Male, J8 Conn_01x02_Male, J9 Conn_01x02_Male, Q1 Q_NMOS_GSD, Q2 Q_NMOS_GSD, U1 Battery_2x18650, U10 HIH-5031, U11 GPS_MTK3339, U2 MAX1719EUT+T, U3 Teensy4.1, U4 TLV2374, U5 TLV2374, U6 MS583702BA01-50, U7 BM1422AGMV-ZE2, U8 MPU-6050-SparkFun, U9 STS21

Commit message: Add files via upload
Parts:
- added C14: 100nF, Capacitor_SMD:C_0805_2012Metric, F.Cu at (184.6, 134.9)
- added C15: 100nF, Capacitor_SMD:C_0805_2012Metric, F.Cu at (197.3, 74.3)
- added C16: 1u, Capacitor_SMD:C_0805_2012Metric_Pad1.18x1.45mm_HandSolder, F.Cu at (159.7, 124.5)
- added C17: 100nF, Capacitor_SMD:C_0805_2012Metric_Pad1.18x1.45mm_HandSolder, F.Cu at (176.9, 125.3)
- added C18: 100nF, Capacitor_SMD:C_0805_2012Metric_Pad1.18x1.45mm_HandSolder, B.Cu at (131.8, 84.8)
- added C19: 100nF, Capacitor_SMD:C_0805_2012Metric_Pad1.18x1.45mm_HandSolder, F.Cu at (127.1, 87.1)
- added C20: 100nF, Capacitor_SMD:C_0805_2012Metric_Pad1.18x1.45mm_HandSolder, B.Cu at (127.1, 87.2)
- added C21: 2.2nF, Capacitor_SMD:C_0805_2012Metric_Pad1.18x1.45mm_HandSolder, B.Cu at (132.9, 82.7)
- added J15: Conn_01x05_Male, Connector_PinHeader_2.54mm:PinHeader_1x05_P2.54mm_Vertical, B.Cu at (100.4, 112.5)
- added J16: Conn_01x05_Male, Connector_PinHeader_2.54mm:PinHeader_1x05_P2.54mm_Vertical, B.Cu at (195.3, 65.2)
- added J17: Conn_01x03_Male, Connector_PinHeader_2.54mm:PinHeader_1x03_P2.54mm_Vertical, F.Cu at (160.5, 137.6)
- added J18: Conn_01x03_Male, Connector_PinHeader_2.54mm:PinHeader_1x03_P2.54mm_Vertical, B.Cu at (126.7, 69.0)
- added J19: Conn_01x07_Male, Connector_PinHeader_2.54mm:PinHeader_1x07_P2.54mm_Vertical, F.Cu at (182.9, 90.6)
- added J20: Conn_01x07_Male, Connector_PinHeader_2.54mm:PinHeader_1x07_P2.54mm_Vertical, B.Cu at (138.5, 79.0)
- added J21: Conn_01x01_Male, Connector_PinHeader_2.54mm:PinHeader_1x01_P2.54mm_Vertical, F.Cu at (177.2, 86.2)
- added J22: Conn_01x01_Male, Connector_PinHeader_2.54mm:PinHeader_1x01_P2.54mm_Vertical, B.Cu at (133.6, 103.3)
- added Q3: Q_NMOS_GSD, Package_TO_SOT_SMD:SOT-23, F.Cu at (121.2, 124.6)
- added Q4: Q_NMOS_GSD, Package_TO_SOT_SMD:SOT-23, F.Cu at (115.0, 121.2)
- added R28: 1M, Resistor_SMD:R_0805_2012Metric_Pad1.20x1.40mm_HandSolder, F.Cu at (121.2, 121.5)
- added R29: R, Resistor_SMD:R_0805_2012Metric_Pad1.20x1.40mm_HandSolder, F.Cu at (117.3, 126.2)
- added R30: 1M, Resistor_SMD:R_0805_2012Metric_Pad1.20x1.40mm_HandSolder, F.Cu at (111.7, 121.2)
- added R31: R, Resistor_SMD:R_0805_2012Metric_Pad1.20x1.40mm_HandSolder, F.Cu at (115.0, 124.1)
- added R32: 47k, Resistor_SMD:R_0805_2012Metric_Pad1.20x1.40mm_HandSolder, B.Cu at (198.0, 71.9)
- added U12: E32_LORA, CanSat:E32_LORA, B.Cu at (108.5, 79.2)
- added U13: HIH-5031, CanSat:HIH-5031-001S, F.Cu at (204.2, 71.2)
- added U14: MPU-6050, Sensor_Motion:InvenSense_QFN-24_4x4mm_P0.5mm, B.Cu at (131.0, 88.5)
- added V1: Vis_M3, CanSat:Vis_M3, F.Cu at (189.9, 137.3)
- added V2: Vis_M3, CanSat:Vis_M3, F.Cu at (153.3, 137.3)
- added V3: Vis_M3, CanSat:Vis_M3, F.Cu at (184.1, 68.8)
- added V4: Vis_M3, CanSat:Vis_M3, F.Cu at (101.0, 137.3)
- added V5: Vis_M3, CanSat:Vis_M3, F.Cu at (137.5, 137.3)
- added V6: Vis_M3, CanSat:Vis_M3, F.Cu at (131.8, 68.8)
- BZ1: footprint CanSat:TSR 2-2450 -> CanSat:KTG1205CL
- C10, C11, C12, C7, C8, C9, J11, J12, J2, J3, J4, J5, J6, L1, R11, R24, R3, R4, R8, R9, U1, U11, U7: moved to B.Cu
- C2: footprint Capacitor_SMD:C_0805_2012Metric -> Capacitor_SMD:CP_Elec_6.3x5.9
- U8: footprint Connector_PinHeader_2.54mm:PinHeader_1x10_P2.54mm_Vertical -> CanSat:MPU6050; moved to B.Cu
- moved R20 337.2 mm to (167.4, 84.7)
- moved R18 336.3 mm to (166.6, 77.1), turned to 90 degrees
- moved R21 332.0 mm to (167.4, 87.2)
- moved R22 326.8 mm to (167.4, 89.7)
- moved J9 326.6 mm to (161.9, 84.7), turned to -90 degrees
- moved R23 324.3 mm to (167.4, 92.2)
- moved R5 322.8 mm to (122.8, 89.6), turned to 90 degrees
- moved BZ1 322.4 mm to (112.2, 70.2), turned to 90 degrees
- moved J10 321.4 mm to (161.9, 87.3), turned to -90 degrees
- moved J8 319.5 mm to (161.9, 82.2), turned to -90 degrees
- moved C6 318.9 mm to (164.4, 134.8), turned to 180 degrees
- moved J13 318.3 mm to (161.9, 89.8), turned to -90 degrees
- moved R27 317.9 mm to (180.0, 88.4), turned to -90 degrees
- moved R19 317.2 mm to (167.4, 82.1)
- moved J7 314.9 mm to (161.9, 79.6), turned to -90 degrees
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Connections:
- C13 pad 1: +3V3 -> VCC
- C13 pad 2: GND -> GND1
- C2 pad 2: GNDA -> GND
- C7 pad 1: +3V3 -> VCC
- C7 pad 2: GND -> GND1
- D1 pad 1: GNDA -> GND
- J1 pad 1: (no net) -> unconnected-(J1-Pad1)
- J1 pad 2: (no net) -> Vin
- J1 pad 3: (no net) -> Net-(J1-Pad3)
- R10 pad 1: Net-(J1-PadNO) -> Net-(J1-Pad3)
- R10 pad 2: GNDA -> GND
- R24 pad 2: GNDA -> GND
- R7 pad 2: GNDA -> GND
- RLA1 pad 1: Net-(J1-PadNO) -> Net-(J1-Pad3)
- RLA1 pad 2: GNDA -> GND
- U1 pad 4: GNDA -> GND
- U3 pad 11: LED3 -> INT
- U3 pad 18: Mes_-5V -> unconnected-(U3-Pad18)
- U3 pad 19: unconnected-(U3-Pad19) -> EN_GPS
- U3 pad 23: AlimNeg -> SigLED3
- U3 pad 24: LED2 -> SigLED2
- U3 pad 30: unconnected-(U3-Pad30) -> Up_Mes_-5V
- U3 pad 35: unconnected-(U3-Pad35) -> DRDY
- U3 pad 36: Photo_1 -> UP_Photo_1
- U3 pad 37: Photo_2 -> UP_Photo_2
- U3 pad 4: unconnected-(U3-Pad4) -> AlimNeg_uP
- U3 pad 42: Photo_3 -> UP_Photo_3
- U3 pad 43: Photo_4 -> UP_Photo_4
- U3 pad 44: Photo_5 -> UP_Photo_5
- U3 pad 45: Photo_6 -> UP_Photo_6
- U4 pad 10: GNDA -> GND
- U4 pad 12: GNDA -> GND
- U4 pad 13: Net-(J10-Pad1) -> Net-(J9-Pad1)
- U4 pad 14: Photo_6 -> Photo_5
- U4 pad 3: GNDA -> GND
- U4 pad 5: GNDA -> GND
- U4 pad 8: Photo_5 -> Photo_6
- U4 pad 9: Net-(J9-Pad1) -> Net-(J10-Pad1)
- U5 pad 1: Photo_2 -> Photo_4
- U5 pad 12: GNDA -> GND
- U5 pad 2: Net-(J14-Pad1) -> Net-(J13-Pad1)
- U5 pad 3: GNDA -> GND
- U5 pad 5: GNDA -> GND
- U5 pad 6: Net-(J13-Pad1) -> Net-(J14-Pad1)
- U5 pad 7: Photo_4 -> Photo_2
- U5 pad 8: VbattTeensy -> Vbatt_conn
- U5 pad 9: VbattTeensy -> Vbatt_conn
- U6 pad 1: +3V3 -> VCC
- U6 pad 2: GND -> GND1
- U6 pad 3: SCL2 -> SCL2_Ext
- U6 pad 4: SDA2 -> SDA2_Ext
- U8 pad 3: INT -> SCL
- U8 pad 4: unconnected-(U8-Pad4) -> SDA
- U8 pad 5: SCL -> SDA1
- U8 pad 6: SDA -> SCL1
- U8 pad 7: +3V3 -> INT
- U8 pad 8: unconnected-(U8-Pad8) -> +3V3
- U9 pad 2: GND -> GND1
- U9 pad 3: SDA2 -> SDA2_Ext
- U9 pad 4: SCL2 -> SCL2_Ext
- U9 pad 5: +3V3 -> VCC
- U9 pad 7: (no net) -> unconnected-(U9-Pad7)
Routing:
- net GND: track 0.00 -> 454.3 mm, vias 0 -> 22
- net +5V: track 0.00 -> 212.3 mm, vias 0 -> 5
- net +3V3: track 0.00 -> 187.2 mm, vias 0 -> 10
- net -5V: track 0.00 -> 137.3 mm, vias 0 -> 3
- net Vin: track 0.00 -> 52.6 mm, vias 0 -> 3
- net GNDA: track 0.00 -> 47.8 mm, vias 0 -> 2
- net GND1: track 0.00 -> 45.7 mm, vias 0 -> 3
- net HMD: track 0.00 -> 43.8 mm, vias 0 -> 1
- net Photo_1: track 0.00 -> 37.8 mm, vias 0 -> 1
- net SDA1: track 0.00 -> 35.0 mm, vias 0 -> 1
- net SDA: track 0.00 -> 33.2 mm, vias 0 -> 2
- net SCL2: track 0.00 -> 32.8 mm, vias 0 -> 1
- net TX_LORA: track 0.00 -> 32.2 mm, vias 0 -> 1
- net SDA2: track 0.00 -> 32.1 mm, vias 0 -> 1
- net SigLED1: track 0.00 -> 31.9 mm, vias 0 -> 1
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- added copper zone on F.Cu, net +3V3
- added copper zone on F.Cu, net +5V
- added copper zone on B.Cu, net -5V
- added copper zone on B.Cu, net GND
- added copper zone on B.Cu, net GND1
- added copper zone on F.Cu, net VCC
Other:
- board outline added: 108.3 x 81.9 mm
- board text added: "CANSAT - PCB batteries 07.03.22 - AB"
- board text added: "CANSAT - PCB principal 14.03.22 - AB"
- board text added: "PCB Ext 07.03.22"
