File: CanSat/CanSat.kicad_sch (KiCad schematic)
At the start: 32 parts, among them J1 XLR3_Switched, J2 Conn_01x04_Male, Q1 Q_NMOS_GSD, Q2 Q_NMOS_GSD, U1 Battery_2x18650, U2 MAX1719EUT+T, U3 Teensy4.1

Commit message: Add files via upload
Parts:
- removed J2: Conn_01x04_Male, Connector_PinHeader_2.54mm:PinHeader_1x04_P2.54mm_Vertical, symbol Connector:Conn_01x04_Male
- removed R1, R2, R4, R5, R8, R9: ${Res_I2C}, Resistor_SMD:R_0805_2012Metric_Pad1.20x1.40mm_HandSolder, symbol Device:R_Small
- added C16: 1u, Capacitor_SMD:C_0805_2012Metric_Pad1.18x1.45mm_HandSolder, symbol Device:C_Small
- added C17: 100nF, Capacitor_SMD:C_0805_2012Metric_Pad1.18x1.45mm_HandSolder, symbol Device:C_Small
- added Q3, Q4: FDN337, Package_TO_SOT_SMD:SOT-23, symbol Device:Q_NMOS_GSD
- added R28, R30: 1M, Resistor_SMD:R_0805_2012Metric_Pad1.20x1.40mm_HandSolder, symbol Device:R
- added R29, R31: R, Resistor_SMD:R_0805_2012Metric_Pad1.20x1.40mm_HandSolder, symbol Device:R
- BZ1: footprint CanSat:TSR 2-2450 -> CanSat:KTG1205CL
- C2: footprint Capacitor_SMD:C_0805_2012Metric -> Capacitor_SMD:CP_Elec_6.3x5.9
- Q1, Q2: value Q_NMOS_GSD -> FDN337
Connections:
- net +5V: now also C16.1, C17.1
- net AlimNeg: no longer U3.23 (31_CTX3)
- net GND: now also C2.2, D1.1 (K), R10.2, R7.2, RLA1.2 (GND), U1.4, C16.2, C17.2, Q3.2 (S), Q4.2 (S), R28.2, R30.2
- net GNDA: no longer C2.2, D1.1 (K), R10.2, R7.2, RLA1.2 (GND), U1.4
- net LED2: now also R29.1; no longer U3.24 (32_OUT1B)
- net LED3: now also R31.1; no longer U3.11 (9_OUT1C)
- net EN_GPS: now reaches U3.19 (27_A13_SCK1)
- net Up_Mes_-5V: now reaches U3.30 (38_CS1_IN1)
- net DRDY: now reaches U3.35 (13_SCK_LED)
- net AlimNeg_uP: now reaches U3.4 (2_OUT2)
- net Mes_-5V: no longer names the net of U3.18 (26_A12_MOSI1)
- net Photo_1 renamed UP_Photo_1
- net Photo_2 renamed UP_Photo_2
- net Photo_3 renamed UP_Photo_3
- net Photo_4 renamed UP_Photo_4
- net Photo_5 renamed UP_Photo_5
- net Photo_6 renamed UP_Photo_6
- new net: Q4.3 (D), R31.2
- new net: Q3.3 (D), R29.2
- new net INT: U3.11 (9_OUT1C)
- new net SigLED2: Q3.1 (G), R28.1, U3.24 (32_OUT1B)
- new net SigLED3: Q4.1 (G), R30.1, U3.23 (31_CTX3)
- no-connect marks 14 -> 15
Other:
- added sheet Autre (Autre.kicad_sch)
- note removed: "Résistances des I2C Valeur : ${Res_I2C} Format : 0805"
