File: CanSat/Photo.kicad_sch (KiCad schematic)
At the start: 31 parts, among them J10 Conn_01x02_Male, J11 Conn_01x02_Male, J12 Conn_01x02_Male, J13 Conn_01x02_Male, J14 Conn_01x02_Male, J3 Conn_01x02_Male, J4 Conn_01x02_Male, J5 Conn_01x02_Male, J6 Conn_01x02_Male, J7 Conn_01x02_Male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

Commit message: Add files via upload
Connections:
- net Photo_2: now also U5.7; no longer U5.1
- net Photo_4: now also U5.1; no longer U5.7
- net Photo_5: now also U4.14; no longer U4.8
- net Photo_6: now also U4.8; no longer U4.14
- net at J14.1 (Pin_1), R23.1: now also U5.6 (2-); no longer U5.2 (2-)
- net at J13.1 (Pin_1), R22.1: now also U5.2 (2-); no longer U5.6 (2-)
- net at J9.1 (Pin_1), R20.1: now also U4.13 (4-); no longer U4.9 (3-)
- net at J10.1 (Pin_1), R21.1: now also U4.9 (3-); no longer U4.13 (4-)
- net GNDA renamed GND
- net VbattTeensy renamed Vbatt_conn
Other:
- moved on the sheet: U4C, U4D, U5A, U5B
