File: CanSat/Sensor.kicad_sch (KiCad schematic)
At the start: 15 parts, among them U10 HIH-5031, U11 GPS_MTK3339, U6 MS583702BA01-50, U7 BM1422AGMV-ZE2, U8 MPU-6050-SparkFun, U9 STS21

Commit message: Add files via upload
Parts:
- added C14, C15: 100nF, Capacitor_SMD:C_0805_2012Metric, symbol Device:C_Small
- added C18, C19, C20: 100nF, Capacitor_SMD:C_0805_2012Metric_Pad1.18x1.45mm_HandSolder, symbol Device:C_Small
- added C21: 2.2nF, Capacitor_SMD:C_0805_2012Metric_Pad1.18x1.45mm_HandSolder, symbol Device:C_Small
- added R32: 47k, Resistor_SMD:R_0805_2012Metric_Pad1.20x1.40mm_HandSolder, symbol Device:R
- added U12: E32_LORA, CanSat:E32_LORA, symbol RF_Module:E32_LORA
- added U13: HIH-5031, CanSat:HIH-5031-001S, symbol Sensor_Humidity:HIH-5031
- added U14: MPU-6050, Sensor_Motion:InvenSense_QFN-24_4x4mm_P0.5mm, symbol Sensor_Motion:MPU-6050
- U8: footprint Connector_PinHeader_2.54mm:PinHeader_1x10_P2.54mm_Vertical -> CanSat:MPU6050
Connections:
- net +3V3: now also U8.8 (AD0), C18.2, C19.1, U14.13 (VDD), U14.8 (VDDIO), U14.9 (AD0); no longer C13.1, C7.1, U6.1 (GND), U8.7 (VIO), U9.5 (VDD)
- net GND: now also R24.2, C14.2, C18.1, C19.2, C20.2, C21.2, U12.7 (GND), U14.1 (CLKIN), U14.11 (FSYNC), U14.18 (GND); no longer C13.2, C7.2, U6.2 (VDD), U9.2 (VSS)
- net GNDA: no longer R24.2
- net INT: now also U8.7 (INT), U14.12 (INT); no longer U8.3 (INT)
- net SCL: now also U8.3 (SCL), U14.23 (SCL); no longer U8.5 (SCL)
- net SCL1: now also U8.6 (ASCL), U14.7 (AUX_SCL); no longer U8.9 (ASCL)
- net SDA: now also U8.4 (SDA), U14.24 (SDA); no longer U8.6 (SDA)
- net SDA1: now also U8.5 (ASDA), U14.6 (AUX_SDA); no longer U8.10 (ASDA)
- net SCL2 renamed SCL2_Ext
- net SDA2 renamed SDA2_Ext
- new net: C20.1, U14.10 (REGOUT)
- new net: C21.1, U14.20 (CPOUT)
- new net +5V: C14.1, U12.6 (Vcc)
- new net AUX_LORA: U12.5 (AUX)
- new net GND1: C13.2, C15.2, C7.2, R32.2, U13.1 (VSS), U6.2 (VDD), U9.2 (VSS)
- new net HMD_Ext: R32.1, U13.2 (VOUT)
- new net M0_LORA: U12.1 (M0)
- new net M1_LORA: U12.2 (M1)
- new net RX_LORA: U12.3 (RxD)
- new net TX_LORA: U12.4 (TxD)
- new net VCC: C13.1, C15.1, C7.1, U13.3 (VDD), U6.1 (GND), U9.5 (VDD)
- no-connect marks 8 -> 6
Other:
- moved on the sheet: C10, C11, C12, C13, C7, C8, C9, L1, R24, U10, U11, U6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
